Commit message: simulation working

File: franka_ros/franka_description/robots/hand.xacro (robot description, xacro)
@@ -74,5 +74,5 @@
       <origin xyz="0 0 0.0584" rpy="0 0 0"/>
       <axis xyz="0 1 0"/>
-      <limit effort="20" lower="0.0" upper="0.04" velocity="0.2"/>
+      <limit effort="0.05" lower="0.0" upper="0.04" velocity="0.2"/>
     </joint>
     <joint name="${ns}_finger_joint2" type="prismatic">
@@ -81,21 +81,14 @@
       <origin xyz="0 0 0.0584" rpy="0 0 0"/>
       <axis xyz="0 -1 0"/>
-      <limit effort="20" lower="0.0" upper="0.04" velocity="0.2"/>
+      <limit effort="0.05" lower="0.0" upper="0.04" velocity="0.2"/>
       <mimic joint="${ns}_finger_joint1" />
     </joint>
-    <!-- <gazebo reference="${ns}_leftfinger">
-      <kp>10000000.0</kp>
-      <kd>1.0</kd>
-      <mu1>100000.0</mu1>
-      <mu2>100000.0</mu2>
-      <minDepth>0.001</minDepth>
+    <gazebo reference="${ns}_leftfinger">
+      <implicitSpringDamper>true</implicitSpringDamper>
+      <cfm>0.1</cfm>
     </gazebo>
     <gazebo reference="${ns}_rightfinger">
-      <kp>10000000.0</kp>
-      <kd>1.0</kd>
-      <mu1>100000.0</mu1>
-      <mu2>100000.0</mu2>
-      <minDepth>0.001</minDepth>
-    </gazebo> -->
+      <cfm>0.1</cfm>
+    </gazebo>
   </xacro:macro>
 </robot>

File: franka_ros/franka_description/robots/panda_arm.xacro (robot description, xacro)
@@ -341,9 +341,9 @@
            <gripper_link> panda_rightfinger </gripper_link>
         </arm>
-       <forces_angle_tolerance>120</forces_angle_tolerance>
-       <update_rate>8</update_rate>
+       <forces_angle_tolerance>100</forces_angle_tolerance>
+       <update_rate>10</update_rate>
        <grip_count_threshold>4</grip_count_threshold>
        <max_grip_count>8</max_grip_count>
-       <release_tolerance>0.003</release_tolerance>
+       <release_tolerance>0.005</release_tolerance>
        <disable_collisions_on_attach>true</disable_collisions_on_attach>
        <contact_topic>__default_topic__</contact_topic>

Commit message: changed gripper open pose

File: franka_ros/franka_description/robots/hand.xacro (robot description, xacro)
@@ -74,5 +74,5 @@
       <origin xyz="0 0 0.0584" rpy="0 0 0"/>
       <axis xyz="0 1 0"/>
-      <limit effort="0.05" lower="0.0" upper="0.04" velocity="0.2"/>
+      <limit effort="0.05" lower="0.0" upper="0.05" velocity="0.2"/>
     </joint>
     <joint name="${ns}_finger_joint2" type="prismatic">
@@ -81,5 +81,5 @@
       <origin xyz="0 0 0.0584" rpy="0 0 0"/>
       <axis xyz="0 -1 0"/>
-      <limit effort="0.05" lower="0.0" upper="0.04" velocity="0.2"/>
+      <limit effort="0.05" lower="0.0" upper="0.05" velocity="0.2"/>
       <mimic joint="${ns}_finger_joint1" />
     </joint>

Commit message: added mug, changed gripper plugin params

File: franka_ros/franka_description/robots/hand.xacro (robot description, xacro)
@@ -74,5 +74,5 @@
       <origin xyz="0 0 0.0584" rpy="0 0 0"/>
       <axis xyz="0 1 0"/>
-      <limit effort="0.05" lower="0.0" upper="0.05" velocity="0.2"/>
+      <limit effort="0.05" lower="0.0" upper="0.04" velocity="0.2"/>
     </joint>
     <joint name="${ns}_finger_joint2" type="prismatic">
@@ -81,5 +81,5 @@
       <origin xyz="0 0 0.0584" rpy="0 0 0"/>
       <axis xyz="0 -1 0"/>
-      <limit effort="0.05" lower="0.0" upper="0.05" velocity="0.2"/>
+      <limit effort="0.05" lower="0.0" upper="0.04" velocity="0.2"/>
       <mimic joint="${ns}_finger_joint1" />
     </joint>
@@ -87,7 +87,11 @@
       <implicitSpringDamper>true</implicitSpringDamper>
       <cfm>0.1</cfm>
+      <minDepth>0.00</minDepth>
+      <maxVel>0</maxVel>
     </gazebo>
     <gazebo reference="${ns}_rightfinger">
       <cfm>0.1</cfm>
+      <minDepth>0.00</minDepth>
+      <maxVel>0</maxVel>
     </gazebo>
   </xacro:macro>

File: franka_ros/franka_description/robots/panda_arm.xacro (robot description, xacro)
@@ -341,9 +341,9 @@
            <gripper_link> panda_rightfinger </gripper_link>
         </arm>
-       <forces_angle_tolerance>100</forces_angle_tolerance>
+       <forces_angle_tolerance>150</forces_angle_tolerance>
        <update_rate>10</update_rate>
-       <grip_count_threshold>4</grip_count_threshold>
+       <grip_count_threshold>1</grip_count_threshold>
        <max_grip_count>8</max_grip_count>
-       <release_tolerance>0.005</release_tolerance>
+       <release_tolerance>0.003</release_tolerance>
        <disable_collisions_on_attach>true</disable_collisions_on_attach>
        <contact_topic>__default_topic__</contact_topic>

Commit message: changed effort limit and object properties

File: franka_ros/franka_description/robots/hand.xacro (robot description, xacro)
@@ -74,5 +74,5 @@
       <origin xyz="0 0 0.0584" rpy="0 0 0"/>
       <axis xyz="0 1 0"/>
-      <limit effort="0.05" lower="0.0" upper="0.04" velocity="0.2"/>
+      <limit effort="1" lower="0.0" upper="0.04" velocity="0.2"/>
     </joint>
     <joint name="${ns}_finger_joint2" type="prismatic">
@@ -81,5 +81,5 @@
       <origin xyz="0 0 0.0584" rpy="0 0 0"/>
       <axis xyz="0 -1 0"/>
-      <limit effort="0.05" lower="0.0" upper="0.04" velocity="0.2"/>
+      <limit effort="1" lower="0.0" upper="0.04" velocity="0.2"/>
       <mimic joint="${ns}_finger_joint1" />
     </joint>

Commit message: grasp fix remove

File: franka_ros/franka_description/robots/hand.xacro (robot description, xacro)
@@ -74,5 +74,5 @@
       <origin xyz="0 0 0.0584" rpy="0 0 0"/>
       <axis xyz="0 1 0"/>
-      <limit effort="1" lower="0.0" upper="0.04" velocity="0.2"/>
+      <limit effort="0.6" lower="0.0" upper="0.04" velocity="0.2"/>
     </joint>
     <joint name="${ns}_finger_joint2" type="prismatic">
@@ -81,5 +81,5 @@
       <origin xyz="0 0 0.0584" rpy="0 0 0"/>
       <axis xyz="0 -1 0"/>
-      <limit effort="1" lower="0.0" upper="0.04" velocity="0.2"/>
+      <limit effort="0.6" lower="0.0" upper="0.04" velocity="0.2"/>
       <mimic joint="${ns}_finger_joint1" />
     </joint>

File: franka_ros/franka_description/robots/panda_arm.xacro (robot description, xacro)
@@ -345,5 +345,5 @@
        <grip_count_threshold>1</grip_count_threshold>
        <max_grip_count>8</max_grip_count>
-       <release_tolerance>0.003</release_tolerance>
+       <release_tolerance>0</release_tolerance>
        <disable_collisions_on_attach>true</disable_collisions_on_attach>
        <contact_topic>__default_topic__</contact_topic>

Commit message: grasp fix remove 2

File: franka_ros/franka_description/robots/hand.xacro (robot description, xacro)
@@ -74,5 +74,5 @@
       <origin xyz="0 0 0.0584" rpy="0 0 0"/>
       <axis xyz="0 1 0"/>
-      <limit effort="0.6" lower="0.0" upper="0.04" velocity="0.2"/>
+      <limit effort="1" lower="0.0" upper="0.04" velocity="0.2"/>
     </joint>
     <joint name="${ns}_finger_joint2" type="prismatic">
@@ -81,5 +81,5 @@
       <origin xyz="0 0 0.0584" rpy="0 0 0"/>
       <axis xyz="0 -1 0"/>
-      <limit effort="0.6" lower="0.0" upper="0.04" velocity="0.2"/>
+      <limit effort="1" lower="0.0" upper="0.04" velocity="0.2"/>
       <mimic joint="${ns}_finger_joint1" />
     </joint>

File: franka_ros/franka_description/robots/panda_arm.xacro (robot description, xacro)
@@ -345,5 +345,5 @@
        <grip_count_threshold>1</grip_count_threshold>
        <max_grip_count>8</max_grip_count>
-       <release_tolerance>0</release_tolerance>
+       <release_tolerance>0.001</release_tolerance>
        <disable_collisions_on_attach>true</disable_collisions_on_attach>
        <contact_topic>__default_topic__</contact_topic>

Commit message: changed grasp plugin config

File: franka_ros/franka_description/robots/hand.xacro (robot description, xacro)
@@ -74,5 +74,5 @@
       <origin xyz="0 0 0.0584" rpy="0 0 0"/>
       <axis xyz="0 1 0"/>
-      <limit effort="1" lower="0.0" upper="0.04" velocity="0.2"/>
+      <limit effort="1" lower="0.0" upper="0.045" velocity="0.2"/>
     </joint>
     <joint name="${ns}_finger_joint2" type="prismatic">
@@ -81,5 +81,5 @@
       <origin xyz="0 0 0.0584" rpy="0 0 0"/>
       <axis xyz="0 -1 0"/>
-      <limit effort="1" lower="0.0" upper="0.04" velocity="0.2"/>
+      <limit effort="1" lower="0.0" upper="0.045" velocity="0.2"/>
       <mimic joint="${ns}_finger_joint1" />
     </joint>

File: franka_ros/franka_description/robots/panda_arm.xacro (robot description, xacro)
@@ -341,9 +341,9 @@
            <gripper_link> panda_rightfinger </gripper_link>
         </arm>
-       <forces_angle_tolerance>150</forces_angle_tolerance>
+       <forces_angle_tolerance>120</forces_angle_tolerance>
        <update_rate>10</update_rate>
        <grip_count_threshold>1</grip_count_threshold>
        <max_grip_count>8</max_grip_count>
-       <release_tolerance>0.001</release_tolerance>
+       <release_tolerance>0.0005</release_tolerance>
        <disable_collisions_on_attach>true</disable_collisions_on_attach>
        <contact_topic>__default_topic__</contact_topic>
